File: atari-st-mod-enhanced-to-standard-joystick-ports-adapter--hardware.kicad_sch (KiCad schematic)
At the start: 50 parts, among them J1 Joy0/Mouse, J2 Joy1, J3 OLED 128×64, J4 Enhanced Joystick Port, J5 Joy0/Mouse, J6 Joy1, Q1 1<Vgsth<2, Low Rdson, Vds >10, Q10 1<Vgsth<2, Low Rdson, Vds >10, Q2 1<Vgsth<2, Low Rdson, Vds >10, Q3 1<Vgsth<2, Low Rdson, Vds >10, Q4 1<Vgsth<2, Low Rdson, Vds >10, Q5 1<Vgsth<2, Low Rdson, Vds >10, Q6 1<Vgsth<2, Low Rdson, Vds >10, Q7 1<Vgsth<2, Low Rdson, Vds >10, Q8 1<Vgsth<2, Low Rdson, Vds >10, Q9 1<Vgsth<2, Low Rdson, Vds >10, SW1 Reset, SW2 Selector, SW3 Activate/Change, SW4 Cancel, U1 LM4040DBZ-3

Commit message: change footprint of J5/J6 for plastic db9 socket
Parts:
- J5, J6: footprint Connector_Dsub:DSUB-9_Female_Horizontal_P2.77x2.84mm_EdgePinOffset4.94mm_Housed_MountingHolesOffset7.48mm -> atari-interconnect:Joystick_Port_DSUB-9_Male_Horizontal_P2.77x2.84mm_EdgePinOffset14.56mm_Housed_MountingHolesOffset8.2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
Changed lines of the file:
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@@
       (effects (font (size 1.27 1.27)))
     )
-    (property "Footprint" "Connector_Dsub:DSUB-9_Female_Horizontal_P2.77x2.84mm_EdgePinOffset4.94mm_Housed_MountingHolesOffset7.48mm" (at 26.67 238.76 0)
+    (property "Footprint" "atari-interconnect:Joystick_Port_DSUB-9_Male_Horizontal_P2.77x2.84mm_EdgePinOffset14.56mm_Housed_MountingHolesOffset8.20mm" (at 26.67 238.76 0)
       (effects (font (size 1.27 1.27)) hide)
     )
@@
       (effects (font (size 1.27 1.27)))
     )
-    (property "Footprint" "Connector_Dsub:DSUB-9_Female_Horizontal_P2.77x2.84mm_EdgePinOffset4.94mm_Housed_MountingHolesOffset7.48mm" (at 74.93 238.76 0)
-      (effects (font (size 1.27 1.27)) hide)
-    )
+    (property "Footprint" "atari-interconnect:Joystick_Port_DSUB-9_Male_Horizontal_P2.77x2.84mm_EdgePinOffset14.56mm_Housed_MountingHolesOffset8.20mm" (at 74.93 238.76 0)
+      (effects (font (size 1.27 1.27)) hide)
+    )
